File: RC Car Module.kicad_sch (KiCad schematic)
At the start: 68 parts, among them J1 USB_C_Receptacle_USB2.0_14P, J2 Conn_01x13, J3 Conn_01x09, J4 Conn_01x02, J6 Conn_01x02, J7 Conn_01x02, J8 Conn_01x04, SW1 SW_Push, SW2 SW_Push, U1 AP62401WU-7, U2 W25Q16JVUXIQ TR, U3 RT6154AGQW, U4 TB6612FNG, U5 RP2040, Y1 12 MHz

Commit message: Began adding radio and made a couple changes to the footprints
Parts:
- added 11111: MBR120VLSFT1G, RP2040:SDO_SOD-123FL_ONS, symbol Schottky_Diodes:MBR120VLSFT1G
- C10, C9: footprint Capacitor_SMD:C_0603_1608Metric -> Capacitor_SMD:C_1206_3216Metric
- L1, L2: footprint Inductor_SMD:L_0201_0603Metric -> easyeda2kicad:IND-SMD_L4.0-W4.0_XAL4030-332MEC
Connections:
- net VSYS: now also 11111.2; no longer 1111.1, C10.1, R10.1, U3.1 (VINA), U3.10 (VIN), U3.11 (VIN)
- new net: 1111.1, 11111.1, C10.1, R10.1, U3.1 (VINA), U3.10 (VIN), U3.11 (VIN)
Other:
- moved on the sheet: C1, C10, C11, C12, C13, C14, C15, C16, C17, C18, C19, C2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

Commit message: Update ReadMe
Parts:
- added D2: LED, LED_SMD:LED_0402_1005Metric, symbol Device:LED
- added R14: 180K, Resistor_SMD:R_0402_1005Metric, symbol Device:R
- added R20: 330, Resistor_SMD:R_0402_1005Metric, symbol Device:R
- C4: renamed from C5; footprint Capacitor_SMD:C_0603_1608Metric -> Capacitor_Tantalum_SMD:CP_EIA-3528-15_AVX-H
- R12: value 180K -> 680K
- R8: value 1M -> 330K
- renumbered 1111 to 111111, 11111 to 1111111, C3 to C1, C11 to C10, C27 to C11, C6 to C14, C14 to C15, C15 to C16, C16 to C17, C17 to C18, C18 to C19, C1 to C2, C19 to C20, C20 to C21, C21 to C22, C22 to C23, C23 to C24, C24 to C25, C25 to C26, C26 to C27, C2 to C3, C4 to C5, C7 to C6, C8 to C7, C9 to C8, C10 to C9, D2 to D1, J6 to J5, J8 to J6, R2 to R1, R14 to R15, R15 to R16, R16 to R17, R17 to R18, R4 to R2, R20 to R21, R21 to R22, R1 to R3, R3 to R4
Connections:
- net GND: now also D2.1 (K), R14.2; no longer R12.2
- net GPIO14: now also R20.1
- net at R12.1, R8.2: no longer U3.3 (FB)
- new net: D2.2 (A), R20.2
- new net: R12.2, R14.1, U3.3 (FB)
Other:
- moved on the sheet: D1, D3, D4, J2, J3, J6, R12, R19, R21, R22, R8

Commit message: Update Readme
Parts:
- removed C27: 0.1uF, Capacitor_SMD:C_0402_1005Metric, symbol Device:C
- removed R12: 680K, Resistor_SMD:R_0402_1005Metric, symbol Device:R
- removed R15: 100K, Resistor_SMD:R_0402_1005Metric, symbol Device:R
- removed R16: 10K, Resistor_SMD:R_0402_1005Metric, symbol Device:R
- removed SW2: SW_Push, Button_Switch_SMD:SW_Push_SPST_NO_Alps_SKRK, symbol Switch:SW_Push
- removed U3: RT6154AGQW, RP2040:QFN_4AGQW_RIT, symbol RT6154A:RT6154AGQW
- added R7: 100K, Resistor_SMD:R_0402_1005Metric, symbol Device:R
- added TP1, TP2, TP3: TestPoint, TestPoint:TestPoint_Pad_1.0x1.0mm, symbol Connector:TestPoint
- added U3: RT6150BGQW, easyeda2kicad:WSON-10_L2.5-W2.5-P0.50-BL-EP, symbol RT6150BGQW:RT6150BGQW
- C4: footprint Capacitor_Tantalum_SMD:CP_EIA-3528-15_AVX-H -> Capacitor_SMD:C_1206_3216Metric
- C6, C7: footprint Capacitor_SMD:C_0603_1608Metric -> Capacitor_SMD:C_1206_3216Metric
- C8: renamed from C9; value 47uF -> 10uF
- C9: renamed from C8; value 47uF -> 22uF
- D1, D2, D3, D4: footprint LED_SMD:LED_0402_1005Metric -> LED_SMD:LED_0805_2012Metric
- L2: footprint easyeda2kicad:IND-SMD_L4.0-W4.0_XAL4030-332MEC -> Inductor_SMD:L_1008_2520Metric
- R9: renamed from R8; value 330K -> 1.02M
- renumbered 111111 to 1111111111111, 1111111 to 11111111111111, C15 to C10, C16 to C11, C17 to C12, C18 to C13, C19 to C14, C20 to C15, C21 to C16, C22 to C17, C23 to C18, C24 to C19, C25 to C20, C26 to C21, C10 to C22, C11 to C23, C12 to C24, C13 to C25, C14 to C26, J4 to J3, J5 to J4, J3 to J5, J7 to J6, J6 to J7, R9 to R10, R14 to R12, R10 to R13, R13 to R14, R17 to R15, R18 to R16, R19 to R17, R20 to R18, R21 to R19, R22 to R20, R7 to R8
Connections:
- net 3V3_EN is gone; now on net GND: R13.2
- net +12V: now also TP1.1
- net +3V3: now also U3.1 (VOUT); no longer U4.19 (STBY)
- net GND: now also U3.11 (EXP), U3.3 (GND), U3.9 (GND)
- net VSYS: now also TP2.1
- net at 1111111111111.1, 11111111111111.1, C8.1: now also R7.1, TP3.1, U3.5 (VIN), U3.8 (VINA); no longer R13.1
- net at L2.1: now also U3.4 (LX1)
- net at L2.2: now also U3.2 (LX2)
- net at R12.1: now also R9.2, U3.10 (FB)
- net STBY: now reaches U5.34 (GPIO22)
- net STBY: now also U4.19 (STBY)
- net GPIO6: now reaches U5.8 (GPIO6)
- net GPIO6: now also J2.6 (Pin_6)
- net GPIO23: no longer names the net of U5.35 (GPIO23)
- net GPIO7: no longer names the net of U5.9 (GPIO7)
- net GPIO7: no longer J2.6 (Pin_6)
- new net: R7.2, U3.6 (EN)
- new net: R13.1, U3.7 (PS)
Other:
- moved on the sheet: C1, C10, C11, C12, C13, C14, C15, C16, C17, C18, C19, C20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
