File: radio/radio.kicad_sch (KiCad schematic)
At the start: 18 parts, among them J1 Conn_02x04_Top_Bottom, U1 NRF24L01, Y1 16mhz

Commit message: Update Readme
Parts:
- added C1: 4.7uF, Capacitor_SMD:C_0402_1005Metric, symbol Device:C
- renumbered C2 to C10, C9 to C2, C8 to C3, C3 to C4, C4 to C5, C5 to C6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
Connections:
- net GND: now also C1.2
- net VDD: now also C1.1
